File: teensy41-m8-din-midi.kicad_pcb (KiCad board)
At the start: 2 copper layers, 62.2 x 35.6 mm, 12 parts, among them J1 IN, J2 OUT, SW1 OUT_CONFIG, SW2 IN_CONFIG, U1 Teensy4.1, U2 6N138

Commit message: Fixed pin assignments
Connections:
- U1 pad 14: unconnected-(U1-12_MISO_MQSL-Pad14) -> MIDI_OUT
- U1 pad 3: MIDI_OUT -> unconnected-(U1-1_TX1_CTX2_MISO1-Pad3)
Routing:
- net MIDI_OUT: track 9.72 -> 24.4 mm
Changed lines of the file:
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@@
       (drillshape 0)
       (scaleselection 1)
-      (outputdirectory "Gerbers/")
+      (outputdirectory "m8-midi/")
     )
   )
@@
   (net 47 "unconnected-(U1-30_CRX3-Pad22)")
   (net 48 "unconnected-(U1-29_TX7-Pad21)")
-  (net 49 "unconnected-(U1-12_MISO_MQSL-Pad14)")
+  (net 49 "unconnected-(U1-1_TX1_CTX2_MISO1-Pad3)")
   (net 50 "unconnected-(U1-3V3-Pad15)")
   (net 51 "unconnected-(U1-24_A10_TX6_SCL2-Pad16)")
@@
       (net 5 "MIDI_IN") (pinfunction "0_RX1_CRX2_CS1") (pintype "bidirectional"))
     (pad "3" thru_hole circle (at -24.13 7.62 180) (size 1.6 1.6) (drill 1.1) (layers "*.Cu" "*.Mask")
-      (net 7 "MIDI_OUT") (pinfunction "1_TX1_CTX2_MISO1") (pintype "bidirectional"))
+      (net 49 "unconnected-(U1-1_TX1_CTX2_MISO1-Pad3)") (pinfunction "1_TX1_CTX2_MISO1") (pintype "bidirectional"))
     (pad "4" thru_hole circle (at -21.59 7.62 180) (size 1.6 1.6) (drill 1.1) (layers "*.Cu" "*.Mask")
       (net 25 "unconnected-(U1-2_OUT2-Pad4)") (pinfunction "2_OUT2") (pintype "bidirectional"))
@@
       (net 34 "unconnected-(U1-11_MOSI_CTX1-Pad13)") (pinfunction "11_MOSI_CTX1") (pintype "bidirectional"))
     (pad "14" thru_hole circle (at 3.81 7.62 180) (size 1.6 1.6) (drill 1.1) (layers "*.Cu" "*.Mask")
-      (net 49 "unconnected-(U1-12_MISO_MQSL-Pad14)") (pinfunction "12_MISO_MQSL") (pintype "bidirectional"))
+      (net 7 "MIDI_OUT") (pinfunction "12_MISO_MQSL") (pintype "bidirectional"))
     (pad "15" thru_hole circle (at 6.35 7.62 180) (size 1.6 1.6) (drill 1.1) (layers "*.Cu" "*.Mask")
       (net 50 "unconnected-(U1-3V3-Pad15)") (pinfunction "3V3") (pintype "power_in"))
@@
   (segment (start 149.4208 91.6358) (end 151.765 93.98) (width 0.25) (layer "F.Cu") (net 6))
   (segment (start 149.4208 80.8408) (end 149.4208 91.6358) (width 0.25) (layer "F.Cu") (net 6))
-  (segment (start 144.145 73.66) (end 146.685 73.66) (width 0.25) (layer "F.Cu") (net 7))
-  (segment (start 146.685 73.66) (end 151.765 78.74) (width 0.25) (layer "F.Cu") (net 7))
+  (segment (start 125.095 80.01) (end 123.825 78.74) (width 0.25) (layer "F.Cu") (net 7))
+  (segment (start 144.145 73.66) (end 140.19 77.615) (width 0.25) (layer "F.Cu") (net 7))
+  (segment (start 139.385991 80.01) (end 125.095 80.01) (width 0.25) (layer "F.Cu") (net 7))
+  (segment (start 140.19 77.615) (end 140.19 79.205991) (width 0.25) (layer "F.Cu") (net 7))
+  (segment (start 140.19 79.205991) (end 139.385991 80.01) (width 0.25) (layer "F.Cu") (net 7))
   (segment (start 130.215 62.865) (end 128.945 61.595) (width 0.25) (layer "F.Cu") (net 66))
   (segment (start 111.65 62.975) (end 111.65 65.655) (width 0.25) (layer "F.Cu") (net 66))
